File: operon.kicad_pcb (KiCad board)
At the start: 2 copper layers, 105 parts, among them P1 USB, P2 CONN_2, P3 MOD_SWD, P4 HEADER1, P5 HEADER2, P6 TC1, P7 TC2, P8 TC3, P9 TC4, Q1 AO3401A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

Commit message: Moved to QFN footprints. Still routing.
Parts:
- removed C12, C13: 1u, CAPC1608N
- added D6: CHRG, LEDC2012N, F.Cu at (146.0, 97.0)
- added R44: 4.7k, RESC1608N, F.Cu at (141.0, 96.0)
- D2: value 1N5819HW -> ESD30V0D3
- U10, U7: value MCP6002-I_MS -> MCP6002-I_MC; footprint MCP6002-I_MS -> MCP6002-I_MC
- U5: value MKL25Z64VLH4 -> MKL25Z64VFM4; footprint MKL25Z64VLH4 -> MKL25Z64VFM4
- U8, U9: value MCP6V02-E_SN -> MCP6V02-E_MD; footprint MCP6V02-E_SN -> MCP6V02-E_MD
- moved R11 238.3 mm to (98.0, 115.0)
- moved R3 232.6 mm to (137.0, 94.0)
- moved R6 228.1 mm to (95.0, 106.0)
- moved R1 224.2 mm to (142.0, 93.0)
- moved R18 223.7 mm to (110.0, 108.0)
- moved R12 216.8 mm to (117.0, 110.0)
- moved R15 216.4 mm to (120.0, 110.0), turned to 180 degrees
- moved R4 215.3 mm to (91.0, 140.0)
- moved C21 213.4 mm to (95.0, 104.0)
- moved R13 207.3 mm to (117.0, 108.0)
- moved R16 205.2 mm to (113.0, 110.0), turned to 180 degrees
- moved R7 204.2 mm to (122.0, 135.0), turned to 90 degrees
- moved C10 204.0 mm to (131.0, 124.0)
- moved C20 201.6 mm to (125.0, 103.0), turned to 180 degrees
- moved R17 195.7 mm to (113.0, 108.0), turned to 180 degrees
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Connections:
- C4 pad 1: N-0000028 -> N-0000033
- C6 pad 1: N-0000027 -> N-0000034
- D2 pad 2: N-0000027 -> N-0000034
- D3 pad 1: /LED -> /GPIO5
- P2 pad 1: N-0000027 -> N-0000034
- P3 pad 2: /SWD_CLK -> /SWD_DIO
- P3 pad 3: /SWD_DIO -> GND
- P3 pad 4: GND -> /SWD_CLK
- R7 pad 2: N-000002 -> N-000001
- R8 pad 2: N-000001 -> N-000002
- S2 pad 1: /BUTTON -> /GPIO4
- U4 pad 1: N-0000027 -> N-0000034
- U4 pad 3: N-0000028 -> N-0000034
- U4 pad 4: (no net) -> N-0000033
- U5 pad 10: /AFE/TC2 -> /SWD_CLK
- U5 pad 11: /AFE/TC3 -> /S1
- U5 pad 12: /AFE/TC4 -> /S2
- U5 pad 13: +3.3VADC -> /SWD_DIO
- U5 pad 14: /AFE/REF -> /GPIO4
- U5 pad 15: GND -> +3.3V
- U5 pad 17: N-0000066 (its old number) -> /CLKIN
- U5 pad 18: /AFE/DAC -> /CLKOUT
- U5 pad 19: N-0000056 (its old number) -> /RESET
- U5 pad 2: N-0000050 -> GND
- U5 pad 20: N-0000051 (its old number) -> /AFE/TC3
- U5 pad 21: N-0000053 -> /AFE/TC4
- U5 pad 22: /SWD_CLK -> /COLD
- U5 pad 23: N-0000047 (its old number) -> /AFE/TC1
- U5 pad 24: N-0000049 -> /GPIO5
- U5 pad 25: /SWD_DIO -> /CS
- U5 pad 26: N-0000059 -> /SCK
- U5 pad 27: N-0000067 -> /MOSI
- U5 pad 28: N-0000054 -> /MISO
- U5 pad 29: N-0000057 -> /GPIO1
- U5 pad 3: +3.3V -> N-000001
- U5 pad 30: +3.3V -> /AFE/TC2
- U5 pad 31: GND -> /GPIO2
- U5 pad 32: /CLKIN -> /GPIO3
- U5 pad 33: /CLKOUT -> GND
- U5 pad 4: GND -> N-000002
- U5 pad 5: N-000002 -> +3.3V
- U5 pad 6: N-000001 -> +5V
- U5 pad 7: +3.3V -> +3.3VADC
- U5 pad 8: +5V -> GND
- U5 pad 9: /AFE/TC1 -> /AFE/DAC
- U6 pad 8: /GPIO6 -> /GPIO4
Routing:
- added copper zone on B.Cu, net GND
- added copper zone on F.Cu, net GND
Other:
- board outline added: 50 x 50 mm
- net class Default: clearance 0.254 -> 0.15; trace_width 0.254 -> 0.15; via_dia 0.889 -> 0.6; via_drill 0.635 -> 0.3
- net class Power added: clearance 0.15, trace_width 0.5, via_dia 0.6, via_drill 0.3
- rule trace_clearance: 0.254 -> 0.15
- rule trace_min: 0.254 -> 0.15
- rule via_min_drill: 0.508 -> 0.3
- rule via_min_size: 0.889 -> 0.6

Commit message: working
Parts:
- removed C21, C6: 1u, CAPC1608N
- removed C4: 10n, CAPC1608N
- removed D2: ESD30V0D3, ESD5V0D3
- removed P2: CONN_2, HEADER350P1X2
- removed R5: 1M, RESC1608N
- removed R6: 510, RESC1608N
- removed U10: MCP6002-I_MC, MCP6002-I_MC
- removed U4: LP2985-50DBVR, LP2985-50DBVR
- added C12: 100n, CAPC1608N, F.Cu at (125.0, 108.0)
- U5: value MKL25Z64VFM4 -> MKL25Z64VFT4; footprint MKL25Z64VFM4 -> MKL25Z64VFT4
- X1: footprint ECS_HC-46X -> OSC-3225
- moved S2 61.6 mm to (145.5, 119.5)
- moved BT1 57.4 mm to (137.5, 146.5), turned to 90 degrees
- moved S1 56.4 mm to (145.5, 113.0)
- moved C14 51.6 mm to (140.0, 120.0)
- moved R1 51.3 mm to (133.0, 143.5), turned to 270 degrees
- moved Q1 50.7 mm to (134.0, 136.0), turned to 90 degrees
- moved R3 49.9 mm to (131.0, 143.5), turned to 270 degrees
- moved U1 49.7 mm to (134.0, 140.0), turned to 180 degrees
- moved C5 48.9 mm to (137.0, 143.5)
- moved D1 48.8 mm to (130.0, 137.0), turned to 270 degrees
- moved C15 45.3 mm to (110.0, 121.0), turned to 180 degrees
- moved L2 45.3 mm to (110.0, 123.0), turned to 180 degrees
- moved R44 44.1 mm to (138.5, 140.0), turned to 90 degrees
- moved D6 40.2 mm to (138.5, 136.5), turned to 90 degrees
- moved C17 37.6 mm to (120.0, 132.5), turned to 270 degrees
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Connections:
- C17 pad 1: +3.3VADC -> +3.3V
- C3 pad 1: N-0000038 -> /VBUS2
- D1 pad 1: N-0000038 -> /VBUS2
- D3 pad 1: /GPIO5 -> /LED
- D6 pad 1: +5V -> /VBUS2
- L1 pad 2: N-0000038 -> /VBUS2
- Q1 pad G: N-0000038 -> /VBUS2
- R15 pad 1: /AFE/TC1_SHIFT -> /AFE/SHIFT1
- R19 pad 1: /AFE/TC2_SHIFT -> /AFE/SHIFT1
- R23 pad 1: /AFE/TC3_SHIFT -> /AFE/SHIFT2
- R27 pad 1: /AFE/TC4_SHIFT -> /AFE/SHIFT2
- R28 pad 2: /AFE/REF -> +3.3VADC
- R3 pad 1: N-0000038 -> /VBUS2
- R30 pad 2: /AFE/REF -> +3.3VADC
- R32 pad 2: /AFE/REF -> +3.3VADC
- R34 pad 2: /AFE/REF -> +3.3VADC
- R7 pad 1: /D+ -> N-0000027
- R7 pad 2: N-000001 (its old number) -> /D+
- R8 pad 1: /D- -> N-0000028
- R8 pad 2: N-000002 -> /D-
- S2 pad 1: /GPIO4 -> /BUTTON
- U1 pad 4: N-0000038 -> /VBUS2
- U5 pad 1: /DAL -> +3.3V
- U5 pad 10: /SWD_CLK -> +3.3VADC
- U5 pad 11: /S1 -> GND
- U5 pad 12: /S2 -> GND
- U5 pad 13: /SWD_DIO -> N-0000038
- U5 pad 14: /GPIO4 -> /AFE/DAC
- U5 pad 15: +3.3V -> N-0000039
- U5 pad 16: GND -> N-0000040
- U5 pad 17: /CLKIN -> /SWD_CLK
- U5 pad 18: /CLKOUT -> /S2
- U5 pad 19: /RESET -> /S1
- U5 pad 20: /AFE/TC3 -> /SWD_DIO
- U5 pad 21: /AFE/TC4 -> /BUTTON
- U5 pad 22: /COLD -> +3.3V
- U5 pad 23: /AFE/TC1 -> GND
- U5 pad 24: /GPIO5 -> /CLKIN
- U5 pad 25: /CS -> /CLKOUT
- U5 pad 26: /SCK -> /RESET
- U5 pad 27: /MOSI -> N-0000041
- U5 pad 28: /MISO -> N-0000033
- U5 pad 29: /GPIO1 -> /AFE/TC3
- U5 pad 3: N-000001 (its old number) -> N-0000027
- U5 pad 30: /AFE/TC2 -> /AFE/TC4
- U5 pad 31: /GPIO2 -> N-0000042
- U5 pad 32: /GPIO3 -> N-0000043
- U5 pad 33: GND -> /COLD
- U5 pad 4: N-000002 -> N-0000028
- U5 pad 7: +3.3VADC -> N-0000036
- U5 pad 8: GND -> N-0000037
- U5 pad 9: /AFE/DAC -> +3.3VADC
- U6 pad 3: /GPIO5 -> /CE
- U6 pad 8: /GPIO4 -> /IRQ
- U7 pad 1: /AFE/TC1_SHIFT -> /AFE/SHIFT1
- U7 pad 2: /AFE/TC1_SHIFT -> /AFE/SHIFT1
- U7 pad 6: /AFE/TC2_SHIFT -> /AFE/SHIFT2
- U7 pad 7: /AFE/TC2_SHIFT -> /AFE/SHIFT2
Routing:
- net +3.3VADC: track 0.00 -> 55.0 mm, vias 0 -> 6
- net /AFE/DAC: track 0.00 -> 27.5 mm, vias 0 -> 2
- net /RESET: track 0.00 -> 21.5 mm
- net /COLD: track 0.00 -> 18.9 mm, vias 0 -> 2
- net /AFE/SHIFT2: track 0.00 -> 17.9 mm, vias 0 -> 2
- net /AFE/SHIFT1: track 0.00 -> 17.6 mm, vias 0 -> 2
- net /BUTTON: track 0.00 -> 16.8 mm, vias 0 -> 2
- net /AFE/TC3: track 0.00 -> 11.0 mm
- net /AFE/TC2: track 0.00 -> 9.82 mm
- net /AFE/TC3-: track 0.00 -> 9.00 mm
- net /AFE/TC1-: track 0.00 -> 9.00 mm
- net /AFE/TC2-: track 0.00 -> 8.76 mm
- net /AFE/TC4-: track 0.00 -> 8.44 mm
- net /AFE/TC3+: track 0.00 -> 7.83 mm
- net /AFE/TC1+: track 0.00 -> 7.71 mm
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Other:
- net class Power: trace_width 0.5 -> 0.3
- board text added: "+"
- board text added: "-"

Commit message: working
Routing:
- net /DAL: track 0.00 -> 24.0 mm
- net /GPIO4: track 0.00 -> 21.4 mm
- net /GPIO3: track 0.00 -> 18.9 mm
- net /GPIO2: track 0.00 -> 18.6 mm
- net /GPIO1: track 0.00 -> 18.3 mm
- net GND: track 4.40 -> 18.6 mm
- net /CE: track 0.00 -> 10.4 mm, vias 0 -> 1
- net +3.3VADC: track 55.0 -> 64.8 mm, vias 6 -> 7
- net /CS: track 0.00 -> 9.35 mm, vias 0 -> 1
- net /IRQ: track 0.00 -> 7.77 mm, vias 0 -> 1
- net /CLKOUT: track 0.00 -> 7.42 mm
- net /CLKIN: track 0.00 -> 6.79 mm
- net /LED: track 0.00 -> 5.67 mm
- net /SHIELD: track 0.00 -> 5.58 mm
- net /SCK: track 0.00 -> 4.34 mm, vias 0 -> 1
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
Commit message: layout done
Parts:
- moved S1 2.50 mm to (145.5, 115.5)
- moved S2 2.50 mm to (145.5, 122.0)
- moved D4 1.00 mm to (142.5, 127.0)
Connections:
- U1 pad 5: (no net) -> N-000003
Routing:
- net /RESET: track 21.5 -> 18.9 mm
- net /BUTTON: track 16.8 -> 17.3 mm
Other:
- board text added: "1"
- board text added: "2"
- board text added: "3"
- board text added: "4"
- board text added: "4x"
- board text added: "RA1"
- board text added: "RA2"
- board text added: "RA3"
