File: operon.kicad_pcb (KiCad board)
At the start: 2 copper layers, 50 x 50 mm, 97 parts, among them P1 USB, P3 MOD_SWD, P4 HEADER1, P5 HEADER2, P6 TC1, P7 TC2, P8 TC3, P9 TC4, Q1 AO3401A, Q2 ZXMN3A01F, Q3 ZXMN3A01F, U1 MCP73831T-2ACI_OT, U2 MCP9700AT-E_LT, U3 IP4221CZ6-S, U5 MKL25Z64VFT4, U6 MOD_NRF24L01, U7 MCP6002-I_MC, U8 MCP6V02-E_MD, U9 MCP6V02-E_MD, X1 HC-46X 16M

Commit message: rerouted
Parts:
- added D2: LED, LEDC2012N, F.Cu at (120.0, 137.5)
- added D7: ZENER, SOD3717X135N, F.Cu at (114.0, 138.0)
- added Q4: ZXMN3A01F, SOT190P230X100-3N, F.Cu at (109.0, 134.0)
- added Q5: ZXMN3A01F, SOT190P230X100-3N, F.Cu at (109.0, 138.0)
- added R5: 100k, RESC1608N, F.Cu at (114.0, 136.0)
- added R6: 100k, RESC1608N, F.Cu at (114.0, 140.0)
- D4, D5: value 1N5819HW -> ZENER
- D6: value CHRG -> ZENER; footprint LEDC2012N -> SOD3717X135N
- moved Q2 30.0 mm to (109.0, 126.0), turned to 180 degrees
- moved Q3 30.0 mm to (109.0, 130.0), turned to 180 degrees
- moved D5 28.7 mm to (114.0, 130.0), turned to 0 degrees
- moved D4 28.5 mm to (114.0, 126.0), turned to 0 degrees
- moved R9 26.5 mm to (114.0, 128.0)
- moved R10 25.0 mm to (114.0, 132.0), turned to 0 degrees
- moved D3 24.7 mm to (138.5, 136.5), turned to 90 degrees
- moved D6 24.6 mm to (114.0, 134.0), turned to 0 degrees
- moved R4 15.6 mm to (120.0, 141.0), turned to 90 degrees
- moved P3 4.50 mm to (138.0, 131.0)
- moved L1 4.03 mm to (122.0, 137.5)
- moved C3 4.00 mm to (124.0, 137.5)
- turned C1 to 270 degrees
Connections:
- D3 pad 1: /LED -> /VBUS2
- D3 pad 2: N-000007 (its old number) -> N-0000010
- D4 pad 2: N-000006 (its old number) -> /FET1
- D5 pad 2: N-000005 -> /FET2
- D6 pad 1: /VBUS2 -> GND
- D6 pad 2: N-0000049 -> /FET3
- P4 pad 1: +5V -> GND
- P4 pad 3: GND -> +5V
- P4 pad 4: /GPIO1 -> /FET1
- P4 pad 5: /GPIO2 -> /FET2
- P4 pad 6: /GPIO3 -> /FET3
- P4 pad 7: /GPIO4 -> /FET4
- P5 pad 1: +5V -> /GPIO1
- P5 pad 2: N-000006 (its old number) -> /GPIO2
- P5 pad 3: N-000005 -> /GPIO3
- Q2 pad D: N-000006 (its old number) -> /FET1
- Q3 pad D: N-000005 -> /FET2
- R4 pad 2: N-000007 (its old number) -> N-0000031
- R44 pad 2: N-0000049 -> N-0000010
- U3 pad 1: /D- -> /D+
- U3 pad 3: /D+ -> /SHIELD
- U3 pad 6: /SHIELD -> /D-
- U5 pad 13: N-0000038 -> /GPIO3
- U5 pad 18: /S2 -> /GPIO2
- U5 pad 19: /S1 -> /GPIO1
- U5 pad 38: /GPIO1 -> /S1
- U5 pad 39: /GPIO2 -> /S2
- U5 pad 40: /CE -> /S3
- U5 pad 46: /GPIO3 -> /CE
- U5 pad 47: /GPIO4 -> /S4
Routing:
- net GND: track 18.6 -> 53.5 mm, vias 0 -> 26
- net +3.3VADC: track 64.8 -> 92.2 mm, vias 7 -> 9
- net /S3: track 0.00 -> 21.8 mm
- net /GPIO4: track 21.4 -> 0.00 mm
- net /GPIO3: track 18.9 -> 0.00 mm
- net /S2: track 2.58 -> 18.6 mm
- net /GPIO2: track 18.6 -> 2.58 mm
- net /GPIO1: track 18.3 -> 2.82 mm
- net /S1: track 2.82 -> 15.4 mm
- net /FET4: track 0.00 -> 10.1 mm
- net /FET3: track 0.00 -> 9.72 mm
- net /FET2: track 0.00 -> 9.52 mm
- net /FET1: track 0.00 -> 9.31 mm
- net /CE: track 10.4 -> 3.11 mm, vias 1 -> 0
- net /S4: track 0.00 -> 6.35 mm
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
Commit message: almost
Routing:
- net +5V: track 0.00 -> 77.4 mm, vias 0 -> 1
- net +3.3V: track 10.6 -> 82.0 mm, vias 0 -> 3
- net /VBUS2: track 0.00 -> 25.3 mm
- net /MOSI: track 5.43 -> 27.5 mm
- net /GPIO1: track 2.82 -> 24.2 mm, vias 0 -> 1
- net /GPIO2: track 2.58 -> 23.9 mm, vias 0 -> 1
- net /GPIO3: track 0.00 -> 20.8 mm
- net /SCK: track 6.43 -> 26.0 mm
- net /D+: track 0.00 -> 16.7 mm, vias 0 -> 2
- net /D-: track 0.00 -> 14.7 mm, vias 0 -> 2
- net /MISO: track 4.85 -> 18.6 mm
- net /SWD_CLK: track 2.20 -> 15.1 mm
- net N-0000023: track 0.00 -> 12.4 mm
- net /VBUS: track 0.00 -> 10.4 mm
- net /SWD_DIO: track 3.74 -> 13.6 mm
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Other:
- board text added: "bharr.is"
- board text added: "operon 0.1"

Commit message: first version
Parts:
- added G***: bharr_copper-front_4mm, bharr_copper-front_4mm, F.Cu at (146.8, 109.5)
- added G***: OSHW_silkscreen-front_4mm, OSHW_silkscreen-front_4mm, F.Cu at (141.5, 139.5)
- added HOLE_M3: Val**, HOLE_M3, F.Cu at (146.0, 104.0)
- added HOLE_M3: Val**, HOLE_M3, F.Cu at (104.0, 104.0)
- added HOLE_M3: Val**, HOLE_M3, F.Cu at (104.0, 146.0)
- added HOLE_M3: Val**, HOLE_M3, F.Cu at (146.0, 146.0)
- moved C10 2.00 mm to (137.0, 127.0)
- moved C7 2.00 mm to (137.0, 125.0)
- moved C8 2.00 mm to (137.0, 123.0)
- moved X1 1.58 mm to (133.5, 124.0)
Routing:
- net /IRQ: track 2.54 -> 31.3 mm
- net /CS: track 4.54 -> 31.4 mm
- net /CE: track 1.98 -> 23.5 mm
- net /S4: track 6.21 -> 26.6 mm, vias 1 -> 2
- net GND: track 61.2 -> 77.4 mm, vias 31 -> 36
- net /MISO: track 18.6 -> 27.3 mm, vias 0 -> 1
- net /GPIO1: track 24.2 -> 21.3 mm
- net /CLKIN: track 6.79 -> 9.38 mm
- net /CLKOUT: track 7.42 -> 9.14 mm
- net /BUTTON: track 17.3 -> 15.7 mm
- net /GPIO2: track 23.9 -> 22.4 mm
- net +3.3V: track 82.0 -> 83.3 mm
- net +5V: track 77.4 -> 76.8 mm
Other:
- board text added: "3.3V"
- board text added: "5V"
- board text added: "CE"
- board text added: "CLK"
- board text added: "CS"
- board text added: "DIO"
- board text added: "DP5050_v1"
- board text added: "GND"
- board text added: "IO"
- board text added: "IO1"
- board text added: "IO2"
- board text added: "IO3"
- board text added: "IRQ"
- board text added: "MISO"
- board text added: "MOSI"
- board text added: "SCK"
- board text added: "operon 0.2"
- board text removed: "operon 0.1"

Commit message: 0.3
Parts:
- renumbered C12 to C1, C25 to C10, C29 to C11, C24 to C12, C28 to C13, C8 to C15, C7 to C16, C15 to C17, C10 to C18, C20 to C2, C17 to C20, C9 to C21, C3 to C22, C1 to C23, C5 to C24, C2 to C25, C11 to C3, C16 to C4, C18 to C5, C22 to C6, C26 to C7, C23 to C8, C27 to C9, R18 to R1, R19 to R11, R16 to R12, R12 to R13, R15 to R14, R27 to R15, R24 to R16, R20 to R17, R23 to R18, R17 to R2, R31 to R21, R30 to R22, R28 to R23, R29 to R24, R35 to R25, R34 to R26, R32 to R27, R33 to R28, R13 to R3, R37 to R30, R41 to R31, R36 to R32, R40 to R33, R39 to R34, R43 to R35, R38 to R36, R42 to R37, R14 to R4, R11 to R40, R9 to R41, R10 to R42, R5 to R43, R6 to R44, R4 to R45, R7 to R46, R8 to R47, R3 to R48, R2 to R49, R26 to R5, R1 to R50, R44 to R51, R25 to R6, R21 to R7, R22 to R8
Other:
- board text added: "R1X"
- board text added: "R2X"
- board text added: "RX"
- board text added: "operon 0.3"
- board text removed: "RA1"
- board text removed: "RA2"
- board text removed: "RA3"
- board text removed: "operon 0.2"

Commit message: Corrected footprint for MCP6V02-E/MD (was 2x3, actually 4x4) Added 'edalm:' prefix to footprints Changed version number to 1.0 (not finalised)
Parts:
- moved U8 0.50 mm to (114.5, 115.0)
Routing:
- net /AFE/TC2+: track 7.27 -> 5.97 mm
- net /AFE/TC4+: track 7.27 -> 6.18 mm
- net /AFE/TC2_OUT: track 7.66 -> 6.60 mm
- net /AFE/TC2-: track 8.76 -> 7.86 mm
- net /AFE/TC4-: track 8.44 -> 7.83 mm
- net /AFE/TC3+: track 7.83 -> 7.28 mm
- net /AFE/TC3_OUT: track 7.45 -> 6.94 mm
Other:
- board text added: "operon 1.0"
- board text removed: "operon 0.3"
